File: LPC-Link2-Board.kicad_pcb (KiCad board)
At the start: 2 copper layers, 75.2 x 49.8 mm, 8 parts, among them J2 CONN_02X05, J3 CONN_02X07, J4 CONN_02X10, J6 CONN_01X09, J7 CONN_02X05, J8 CONN_02X10, J9 CONN_02X12

Commit message: Rev1
Parts:
- added G***: LOGO, logo:logo_F_Cu_h2.3, F.Cu at (146.8, 107.0)
